File: Macropad-3x4.kicad_pcb (KiCad board)
At the start: 2 copper layers, 42 parts, among them SW1 RotaryEncoder_Switch, SW2 RotaryEncoder_Switch, U1 ProMicro

Commit message: begin placing components on pcb
Parts:
- moved D9 334.4 mm to (54.0, 90.5), turned to 90 degrees
- moved D5 329.9 mm to (54.0, 71.4), turned to 90 degrees
- moved D10 315.5 mm to (73.0, 90.5), turned to 90 degrees
- moved D6 311.2 mm to (73.0, 71.4), turned to 90 degrees
- moved D2 308.2 mm to (73.0, 52.4), turned to 90 degrees
- moved D11 296.7 mm to (92.1, 90.4), turned to 90 degrees
- moved D7 292.7 mm to (92.1, 71.4), turned to 90 degrees
- moved D3 290.1 mm to (92.1, 52.4), turned to 90 degrees
- moved D12 277.9 mm to (111.1, 90.4), turned to 90 degrees
- moved D8 274.3 mm to (111.1, 71.4), turned to 90 degrees
- moved D4 272.1 mm to (111.1, 52.4), turned to 90 degrees
- moved D1 6.35 mm to (54.0, 52.4)
Routing:
- net Net-(D10-K): track 0.00 -> 57.2 mm
- net Net-(D5-K): track 0.00 -> 57.1 mm
- net Net-(D1-K): track 0.00 -> 57.1 mm
- net Net-(D8-A): track 0.00 -> 6.87 mm
- net Net-(D7-A): track 0.00 -> 6.87 mm
- net Net-(D6-A): track 0.00 -> 6.87 mm
- net Net-(D5-A): track 0.00 -> 6.87 mm
- net Net-(D4-A): track 0.00 -> 6.87 mm
- net Net-(D3-A): track 0.00 -> 6.87 mm
- net Net-(D2-A): track 0.00 -> 6.87 mm
- net Net-(D1-A): track 0.00 -> 6.87 mm
- net Net-(D9-A): track 0.00 -> 6.87 mm
- net Net-(D10-A): track 0.00 -> 6.87 mm
- net Net-(D12-A): track 0.00 -> 6.81 mm
- net Net-(D11-A): track 0.00 -> 6.81 mm
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